File: Hardware/PCB/v0.2/openhandheld-mx.kicad_pcb (KiCad board)
At the start: 4 copper layers, 84 x 42 mm, 112 parts, among them J1 TYPE-C-31-M-12, J2 SJ-3524-SMT-TR, J3 Battery, J4 1040310811, J5 PPPC062LFBN-RC, Q1 SI2102-TP, Q2 SI2102-TP, Q3 SI2102-TP, Q4 SI2101-TP, Q5 SI2102-TP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

Commit message: PCB v0.2: Silkscreen.
Parts:
- added REF**: OSHW-Logo_7.5x8mm_SilkScreen, Symbol:OSHW-Logo_7.5x8mm_SilkScreen, B.Cu at (25.5, -5.15)
- SW3: value A -> B
- SW4: value B -> A
- moved R34 17.5 mm to (4.20, -1.75)
- moved R33 16.2 mm to (5.20, -1.75)
Connections:
- D1 pad 5: (no net) -> Net-(D1-Pad5)
- D1 pad 6: (no net) -> Net-(D1-Pad6)
- J1 pad A8: (no net) -> Net-(J1-PadA8)
- J1 pad B8: (no net) -> Net-(J1-PadB8)
- J4 pad 1: (no net) -> Net-(J4-Pad1)
- J4 pad 10: (no net) -> Net-(J4-Pad10)
- J4 pad 8: (no net) -> Net-(J4-Pad8)
- J4 pad 9: (no net) -> Net-(J4-Pad9)
- R33 pad 1: /BTN_A -> /BTN_B
- R34 pad 1: /BTN_B -> /BTN_A
- SW3 pad 1: /BTN_A -> /BTN_B
- SW4 pad 1: /BTN_B -> /BTN_A
- U10 pad 11: (no net) -> Net-(U10-Pad11)
- U10 pad 12: (no net) -> Net-(U10-Pad12)
- U11 pad 4: (no net) -> Net-(U11-Pad4)
- U2 pad 1: (no net) -> Net-(U2-Pad1)
- U2 pad 10: (no net) -> Net-(U2-Pad10)
- U2 pad 11: (no net) -> Net-(U2-Pad11)
- U2 pad 12: (no net) -> Net-(U2-Pad12)
- U2 pad 15: (no net) -> Net-(U2-Pad15)
- U2 pad 16: (no net) -> Net-(U2-Pad16)
- U2 pad 17: (no net) -> Net-(U2-Pad17)
- U2 pad 18: (no net) -> Net-(U2-Pad18)
- U2 pad 22: (no net) -> Net-(U2-Pad22)
- U2 pad 24: (no net) -> Net-(U2-Pad24)
- U6 pad 1: (no net) -> Net-(U6-Pad1)
- U6 pad 4: (no net) -> Net-(U6-Pad4)
- U6 pad 5: (no net) -> Net-(U6-Pad5)
- U7 pad 4: (no net) -> Net-(U7-Pad4)
- U7 pad 7: (no net) -> Net-(U7-Pad7)
- U8 pad 2: /BTN_A -> /BTN_B
- U8 pad 3: /BTN_B -> /BTN_A
Routing:
- net /BTN_B: track 88.4 -> 51.3 mm
- net /BTN_A: track 71.2 -> 64.2 mm
- net /EN: track 36.3 -> 42.8 mm
- net GND: track 127.9 -> 126.7 mm, vias 64 -> 106
- net /SPI2_MISO: track 97.1 -> 98.1 mm
Other:
- board text added: "+"
- board text added: "-"
- board text added: "1"
- board text added: "2"
- board text added: "3"
- board text added: "4"
- board text added: "A"
- board text added: "B"
- board text added: "MX"
- board text added: "OpenHandheld"
- board text added: "X"
- board text added: "Y"
- board text added: "Z"
- board text added: "openhandheld.com"
- board text added: "v0.2"
- board text added: "©2020 Alfonso Luna Licensed under CERN OHL v1.2"

Commit message: Case v0.2: Finished
Changed lines of the file:
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@@
   (general
     (thickness 1.6)
-    (drawings 122)
+    (drawings 121)
     (tracks 1506)
     (zones 0)
@@
   (page A4)
   (layers
-    (0 F.Cu signal hide)
+    (0 F.Cu signal)
     (1 In1.Cu power hide)
     (2 In2.Cu power hide)
-    (31 B.Cu signal hide)
+    (31 B.Cu signal)
     (32 B.Adhes user hide)
     (33 F.Adhes user hide)
     (34 B.Paste user hide)
     (35 F.Paste user hide)
-    (36 B.SilkS user)
-    (37 F.SilkS user hide)
+    (36 B.SilkS user hide)
+    (37 F.SilkS user)
     (38 B.Mask user hide)
-    (39 F.Mask user hide)
+    (39 F.Mask user)
     (40 Dwgs.User user hide)
     (41 Cmts.User user hide)
@@
       (drillshape 0)
       (scaleselection 1)
-      (outputdirectory "../../../../../home/alfonso/Desktop/Gerbers"))
+      (outputdirectory "/home/alfonso/Desktop/Gerbers/"))
   )
   (net 0 "")
@@
   (module _AKL_Optical:Vishay_IR locked (layer B.Cu)
     (at 10.5 -20 90)
+    (attr smd)
     (fp_text reference D5 (at 0 2.75 90) (layer B.SilkS) hide
       (effects (font (size 1 1) (thickness 0.15)) (justify mirror))
@@
   (module _AKL_Optical:Vishay_IR locked (layer B.Cu)
     (at -10.5 -20 90)
+    (attr smd)
     (fp_text reference D6 (at 0 2.75 90) (layer B.SilkS) hide
       (effects (font (size 1 1) (thickness 0.15)) (justify mirror))
@@
   (module _AKL_Optical:150044M155260 locked (layer B.Cu)
     (at -37.25 -3.25)
+    (attr smd)
     (fp_text reference D7 (at 0 1.7) (layer B.SilkS) hide
       (effects (font (size 1 1) (thickness 0.15)) (justify mirror))
@@
   (module _AKL_IC:DSC60XX-3.2x2.5 (layer B.Cu)
     (at -9.7 5.9 90)
+    (attr smd)
     (fp_text reference U5 (at 0 2.5 90) (layer B.SilkS) hide
       (effects (font (size 1 1) (thickness 0.15)) (justify mirror))
@@
     )
   )
-  (gr_text openhandheld.com (at -28.15 17.15) (layer F.SilkS)
-    (effects (font (size 0.75 0.75) (thickness 0.15) italic))
-  )
   (gr_text - (at 25.25 14) (layer B.SilkS)
     (effects (font (size 1 1) (thickness 0.25)) (justify mirror))
@@
     (effects (font (size 0.75 0.75) (thickness 0.15) italic) (justify mirror))
   )
-  (gr_text v0.2 (at 25.5 -9) (layer F.SilkS)
+  (gr_text v0.2 (at 25.5 -9.05) (layer F.SilkS)
     (effects (font (size 0.75 0.75) (thickness 0.15)))
   )
@@
     (effects (font (size 1.25 1.25) (thickness 0.25) italic))
   )
-  (gr_line (start -35.5 14.5) (end -37 16) (layer F.SilkS) (width 0.15))
-  (gr_poly (pts (xy -35.25 14.25) (xy -35.25 14.957107) (xy -35.957107 14.25)) (layer F.SilkS) (width 0.1))
-  (gr_poly (pts (xy -37 18.5) (xy -37.5 18) (xy -36.5 18)) (layer F.SilkS) (width 0.1))
-  (gr_poly (pts (xy -34.5 16) (xy -35 16.5) (xy -35 15.5)) (layer F.SilkS) (width 0.1))
-  (gr_text Z (at -34.5 13.5) (layer F.SilkS)
+  (gr_line (start -37.7 13.7) (end -39.2 15.2) (layer F.SilkS) (width 0.15))
+  (gr_poly (pts (xy -37.45 13.45) (xy -37.45 14.157107) (xy -38.157107 13.45)) (layer F.SilkS) (width 0.1))
+  (gr_poly (pts (xy -39.2 17.7) (xy -39.7 17.2) (xy -38.7 17.2)) (layer F.SilkS) (width 0.1))
+  (gr_poly (pts (xy -36.7 15.2) (xy -37.2 15.7) (xy -37.2 14.7)) (layer F.SilkS) (width 0.1))
+  (gr_text Z (at -36.7 12.7) (layer F.SilkS)
     (effects (font (size 0.75 0.75) (thickness 0.15)))
   )
-  (gr_text Y (at -37 19.25) (layer F.SilkS)
+  (gr_text Y (at -39.2 18.45) (layer F.SilkS)
     (effects (font (size 0.75 0.75) (thickness 0.15)))
   )
-  (gr_text X (at -33.75 16) (layer F.SilkS)
+  (gr_text X (at -35.95 15.2) (layer F.SilkS)
     (effects (font (size 0.75 0.75) (thickness 0.15)))
   )
-  (gr_line (start -37 16) (end -35 16) (layer F.SilkS) (width 0.15))
-  (gr_line (start -37 16) (end -37 18) (layer F.SilkS) (width 0.15))
+  (gr_line (start -39.2 15.2) (end -37.2 15.2) (layer F.SilkS) (width 0.15))
+  (gr_line (start -39.2 15.2) (end -39.2 17.2) (layer F.SilkS) (width 0.15))
   (gr_arc (start 10.5 -20) (end 9.9 -19.4) (angle -90) (layer F.SilkS) (width 0.15))
   (gr_circle (center 10.5 -20) (end 10.501 -20) (layer F.SilkS) (width 0.15))
@@
   (segment (start -18.650001 13.95) (end -18.650001 13.450001) (width 0.15) (layer B.Cu) (net 61))
   (segment (start -18.05 12.85) (end -18.05 11.55) (width 0.15) (layer B.Cu) (net 61))
+  (segment (start 36.25 -7.05) (end 36.25 2.05) (width 0.15) (layer F.Cu) (net 62))
+  (via (at -9.100003 3.1) (size 0.6) (drill 0.3) (layers F.Cu B.Cu) (net 62))
+  (segment (start -9.55 2.650003) (end -9.55 1.7875) (width 0.15) (layer B.Cu) (net 62))
+  (segment (start -9.100003 3.1) (end -9.55 2.650003) (width 0.15) (layer B.Cu) (net 62))
+  (via (at 36.25 -8.55) (size 0.6) (drill 0.3) (layers F.Cu B.Cu) (net 62))
+  (segment (start 36.25 -7.05) (end 36.25 -8.55) (width 0.15) (layer F.Cu) (net 62))
+  (via (at 4.2 -0.45) (size 0.6) (drill 0.3) (layers F.Cu B.Cu) (net 62))
+  (segment (start 4.35001 -0.44999) (end 4.35 -0.45) (width 0.15) (layer B.Cu) (net 62))
+  (segment (start -8.097999 3.625001) (end -8.575002 3.625001) (width 0.15) (layer F.Cu) (net 62))
+  (segment (start -7.824999 3.352001) (end -8.097999 3.625001) (width 0.15) (layer F.Cu) (net 62))
+  (segment (start -7.42503 2.72503) (end -7.824999 3.124999) (width 0.15) (layer F.Cu) (net 62))
+  (segment (start 0.849245 2.72503) (end -7.42503 2.72503) (width 0.15) (layer F.Cu) (net 62))
+  (segment (start -8.575002 3.625001) (end -9.100003 3.1) (width 0.15) (layer F.Cu) (net 62))
+  (segment (start 3.724276 -0.150001) (end 0.849245 2.72503) (width 0.15) (layer F.Cu) (net 62))
+  (segment (start -7.824999 3.124999) (end -7.824999 3.352001) (width 0.15) (layer F.Cu) (net 62))
+  (segment (start 4.2 -0.45) (end 4.2 -1.265) (width 0.15) (layer B.Cu) (net 62))
+  (segment (start 28.14999 -0.44999) (end 36.25 -8.55) (width 0.15) (layer B.Cu) (net 62))
+  (segment (start 3.900001 -0.150001) (end 3.724276 -0.150001) (width 0.15) (layer F.Cu) (net 62))
+  (segment (start 4.2 -0.45) (end 3.900001 -0.150001) (width 0.15) (layer F.Cu) (net 62))
+  (segment (start 4.2 -0.45) (end 4.79498 0.14498) (width 0.15) (layer B.Cu) (net 62))
+  (segment (start 27.55502 0.14498) (end 28.14999 -0.44999) (width 0.15) (layer B.Cu) (net 62))
+  (segment (start 4.79498 0.14498) (end 27.55502 0.14498) (width 0.15) (layer B.Cu) (net 62))
   (segment (start 26.25 -2.05) (end 26.25 7.05) (width 0.15) (layer F.Cu) (net 63))
   (via (at -8.35 3.1) (size 0.6) (drill 0.3) (layers F.Cu B.Cu) (net 63))
@@
   (segment (start 5.99497 -0.15503) (end 22.85503 -0.15503) (width 0.15) (layer B.Cu) (net 63))
   (segment (start 23.25 -0.55) (end 23.6 -0.9) (width 0.15) (layer B.Cu) (net 63))
-  (segment (start 36.25 -7.05) (end 36.25 2.05) (width 0.15) (layer F.Cu) (net 62))
-  (via (at -9.100003 3.1) (size 0.6) (drill 0.3) (layers F.Cu B.Cu) (net 62))
-  (segment (start -9.55 2.650003) (end -9.55 1.7875) (width 0.15) (layer B.Cu) (net 62))
-  (segment (start -9.100003 3.1) (end -9.55 2.650003) (width 0.15) (layer B.Cu) (net 62))
-  (via (at 36.25 -8.55) (size 0.6) (drill 0.3) (layers F.Cu B.Cu) (net 62))
-  (segment (start 36.25 -7.05) (end 36.25 -8.55) (width 0.15) (layer F.Cu) (net 62))
-  (via (at 4.2 -0.45) (size 0.6) (drill 0.3) (layers F.Cu B.Cu) (net 62))
-  (segment (start 4.35001 -0.44999) (end 4.35 -0.45) (width 0.15) (layer B.Cu) (net 62))
-  (segment (start -8.097999 3.625001) (end -8.575002 3.625001) (width 0.15) (layer F.Cu) (net 62))
-  (segment (start -7.824999 3.352001) (end -8.097999 3.625001) (width 0.15) (layer F.Cu) (net 62))
-  (segment (start -7.42503 2.72503) (end -7.824999 3.124999) (width 0.15) (layer F.Cu) (net 62))
-  (segment (start 0.849245 2.72503) (end -7.42503 2.72503) (width 0.15) (layer F.Cu) (net 62))
-  (segment (start -8.575002 3.625001) (end -9.100003 3.1) (width 0.15) (layer F.Cu) (net 62))
-  (segment (start 3.724276 -0.150001) (end 0.849245 2.72503) (width 0.15) (layer F.Cu) (net 62))
-  (segment (start -7.824999 3.124999) (end -7.824999 3.352001) (width 0.15) (layer F.Cu) (net 62))
-  (segment (start 4.2 -0.45) (end 4.2 -1.265) (width 0.15) (layer B.Cu) (net 62))
-  (segment (start 28.14999 -0.44999) (end 36.25 -8.55) (width 0.15) (layer B.Cu) (net 62))
-  (segment (start 3.900001 -0.150001) (end 3.724276 -0.150001) (width 0.15) (layer F.Cu) (net 62))
-  (segment (start 4.2 -0.45) (end 3.900001 -0.150001) (width 0.15) (layer F.Cu) (net 62))
-  (segment (start 4.2 -0.45) (end 4.79498 0.14498) (width 0.15) (layer B.Cu) (net 62))
-  (segment (start 27.55502 0.14498) (end 28.14999 -0.44999) (width 0.15) (layer B.Cu) (net 62))
-  (segment (start 4.79498 0.14498) (end 27.55502 0.14498) (width 0.15) (layer B.Cu) (net 62))
   (segment (start 11.485 19.985) (end 11.7 20.2) (width 0.15) (layer B.Cu) (net 64))
   (segment (start 13.163999 19.699999) (end 12.643998 20.22) (width 0.15) (layer B.Cu) (net 64))
