File: Hardware/PCB/v0.2/openhandheld-mx.sch (KiCad schematic (older format))
At the start: 0 parts

Commit message: PCB v0.2: Completed schematic
Parts:
- added C1, C13, C14, C17, C20, C23, C26, C28, C7: 10uF, Capacitor_SMD:C_0805_2012Metric, symbol _AKL_Capacitor:10uF
- added C10, C16, C9: 1uF, Capacitor_SMD:C_0603_1608Metric, symbol _AKL_Capacitor:1uF
- added C11, C12, C15, C19, C2, C21, C22, C24, C25, C27, C29, C3, C4, C5, C8: 100nF, Capacitor_SMD:C_0603_1608Metric, symbol _AKL_Capacitor:100nF
- added C18, C6: 100uF, Capacitor_SMD:C_1210_3225Metric, symbol _AKL_Capacitor:100uF
- added D1: PESD5V0L5UY, Package_TO_SOT_SMD:SOT-363_SC-70-6, symbol _AKL_Diode:PESD5V0L5UY
- added D2, D3: BLUE, LED_SMD:LED_0603_1608Metric, symbol _AKL_Optical:150060BS75000
- added D4: RED, LED_SMD:LED_0603_1608Metric, symbol _AKL_Optical:150060SS75000
- added D5: VEMD10940F, _AKL_Optical:Vishay_IR, symbol _AKL_Optical:VEMD10940F
- added D6: VSMB10940, _AKL_Optical:Vishay_IR, symbol _AKL_Optical:VSMB10940
- added D7: RGB, _AKL_Optical:150044M155260, symbol _AKL_Optical:150044M155260
- added D8: MBR0520L, Diode_SMD:D_SOD-123, symbol _AKL_Diode:MBR0520L
- added D9: GREEN, LED_SMD:LED_0603_1608Metric, symbol _AKL_Optical:150060VS75000
- added DS1: ST7789_1.54_240x240, _AKL_Display:ST7789_1.54_240x240, symbol _AKL_Display:ST7789_1.54_240x240
- added J1: TYPE-C-31-M-12, Connector_USB:USB_C_Receptacle_HRO_TYPE-C-31-M-12, symbol _AKL_Connector:TYPE-C-31-M-12
- added J2: SJ-3524-SMT-TR, _AKL_Connector:SJ-3524-SMT-TR, symbol _AKL_Connector:SJ-3524-SMT-TR
- added J3: BK-880, _AKL_Battery:BK-880, symbol _AKL_Battery:BK-880
- added J4: 1040310811, Connector_Card:microSD_HC_Molex_104031-0811, symbol _AKL_Connector:1040310811
- added J5: PPPC062LFBN-RC, Connector_PinSocket_2.54mm:PinSocket_2x06_P2.54mm_Vertical, symbol _AKL_Connector:PPPC062LFBN-RC
- added LS1: CMS-151135-078S, _AKL_Speaker:Speaker_15x11mm, symbol _AKL_Speaker:CMS-151135-078S
- added Q1, Q2, Q3, Q5: FDN327N, Package_TO_SOT_SMD:SOT-23, symbol _AKL_Transistor:FDN327N
- added Q4: FDN340P, Package_TO_SOT_SMD:SOT-23, symbol _AKL_Transistor:FDN340P
- added R1, R10, R16, R2, R26, R29, R30, R33, R34, R35, R38, R6, R7: 20K, Resistor_SMD:R_0603_1608Metric, symbol _AKL_Resistor:20K
- added R11, R12, R13, R23: 1K8, Resistor_SMD:R_0603_1608Metric, symbol _AKL_Resistor:1K8
- added R14, R21: 2K4, Resistor_SMD:R_0603_1608Metric, symbol _AKL_Resistor:2K4
- added R15, R25, R37, R40: 120K, Resistor_SMD:R_0603_1608Metric, symbol _AKL_Resistor:120K
- added R17, R19, R27, R28, R4, R5: 5K1, Resistor_SMD:R_0603_1608Metric, symbol _AKL_Resistor:5K1
- added R18: 150, Resistor_SMD:R_0603_1608Metric, symbol _AKL_Resistor:150
- added R20, R32: 510, Resistor_SMD:R_0603_1608Metric, symbol _AKL_Resistor:510
- added R22, R8: 240, Resistor_SMD:R_0603_1608Metric, symbol _AKL_Resistor:240
- added R24, R3: 1K, Resistor_SMD:R_0603_1608Metric, symbol _AKL_Resistor:1K
- added R31, R9: 100, Resistor_SMD:R_0603_1608Metric, symbol _AKL_Resistor:100
- added R36, R39: 75K, Resistor_SMD:R_0603_1608Metric, symbol _AKL_Resistor:75K
- added SW1: RESET, _AKL_Switch:EVQPU, symbol _AKL_Switch:EVQ-PUL02K
- added SW2: ON/OFF, _AKL_Switch:CUS-12TB, symbol _AKL_Switch:CUS-12TB
- added SW3: A, _AKL_Switch:TL3301TF160QG, symbol _AKL_Switch:TL3301TF160QG
- added SW4: B, _AKL_Switch:TL3301TF160QG, symbol _AKL_Switch:TL3301TF160QG
- added SW5: START, _AKL_Switch:EVQPU, symbol _AKL_Switch:EVQ-PUL02K
- added SW6: SELECT, _AKL_Switch:EVQPU, symbol _AKL_Switch:EVQ-PUL02K
- added U1: TLV9061IDBVR, Package_TO_SOT_SMD:SOT-23-5, symbol _AKL_IC:TLV9061IDBVR
- added U10: LIS2DE12TR, Package_LGA:LGA-12_2x2mm_P0.5mm, symbol _AKL_IC:LIS2DE12TR
- added U11: TLV74333PDBVR, Package_TO_SOT_SMD:SOT-23-5, symbol _AKL_IC:TLV74333PDBVR
- added U2: CP2102N-A02-GQFN24, Package_DFN_QFN:QFN-24-1EP_4x4mm_P0.5mm_EP2.6x2.6mm, symbol _AKL_IC:CP2102N-A02-GQFN24
- added U3: MCP73831T-2ACI_OT, Package_TO_SOT_SMD:SOT-23-5, symbol _AKL_IC:MCP73831T-2ACI_OT
- added U4: PAM8301AAF, Package_TO_SOT_SMD:SOT-23-6, symbol _AKL_IC:PAM8301AAF
- added U5: DSC6001CI1A-008.0000T, _AKL_IC:DSC60XX-3.2x2.5, symbol _AKL_IC:DSC6001CI1A-008.0000T
- added U6: VSOP38338, _AKL_IC:VSOP38338, symbol _AKL_IC:VSOP38338
- added U7: AP9211S-AN-HAC-7, _AKL_IC:AP9211S-AN-HAC-7, symbol _AKL_IC:AP9211S-AN-HAC-7
- added U8: STM32L431CCU6, _AKL_IC:STM32-UFQFPN48, symbol _AKL_IC:STM32L431CCU6
- added U9: W25Q64JVZPIQ, Package_SON:WSON-8-1EP_6x5mm_P1.27mm_EP3.4x4.3mm, symbol _AKL_IC:W25Q64JVZPIQ
- added VR1: FJ08K-N, _AKL_ResistorVar:FJ08K-N, symbol _AKL_ResistorVar:FJ08K-N
Connections:
- new net 3V3: C1.1, C10.1, C11.1, C12.1, C13.1, C15.1, C17.1, C19.1, C2.1, C20.1, C21.1, C23.1, C24.1, C25.1, C27.1, C28.1, C29.1, C3.1, C9.1, D7.1 (A), DS1.3 (LEDA), DS1.4 (VDD), J4.4 (VDD), J5.2 (Pin_2), R10.1, R11.1, R13.1, R17.1, R19.1, R26.1, R27.1, R28.1, R29.1, R3.1, R32.1, R6.1, R7.1, SW3.2, SW4.2, SW5.2, SW6.2, U1.5 (V+), U10.10 (VDD_IO), U10.2 (CS), U10.3 (SDO/SA0), U10.9 (VDD), U11.5 (OUT), U2.5 (VIO), U2.6 (VDD), U2.7 (VREGIN), U4.4 (~SD), U5.1 (OE), U5.4 (VDD), U6.2 (VS), U8.1 (VBAT), U8.24 (VDD), U8.36 (VDD), U8.48 (VDD), U8.9 (VDDA/VREF+), U9.8 (VCC), VR1.1 (X+), VR1.4 (+Y)
- new net AP9_VDD: C22.1, R20.2, U7.3 (VDD)
- new net AUD1: R8.2, U1.1, U1.4 (-)
- new net AUD2: C5.1, C6.2, R8.1, R9.1
- new net AUD3: C6.1, J2.R, J2.T, R12.1
- new net AUD4: C8.1, J2.TN
- new net AUD5: C8.2, R15.2
- new net AUD6: R15.1, U4.3 (IN)
- new net BAT_GND: C22.2, J3.2 (-), U7.1 (S1), U7.2 (VSS)
- new net BOOT: Q1.3 (D), Q3.1 (G), R6.2
- new net BOOT0: Q3.3 (D), R10.2, U8.44 (PH3/BOOT0)
- new net BTN_A: R33.1, SW3.1, U8.2 (PC13)
- new net BTN_B: R34.1, SW4.1, U8.3 (PC14/OSC32_IN)
- new net BTN_SELECT: R38.1, SW6.1, U8.6 (PH1/OSC_OUT)
- new net BTN_START: R35.1, SW5.1, U8.4 (PC15/OSC32_OUT)
- new net CC1: J1.A5 (CC1), R5.1
- new net CC2: J1.B5 (CC2), R4.1
- new net CHG_STAT: D4.1 (K), U3.1 (STAT)
- new net DAC_PWM_OUT: U1.3 (+), U8.15 (PA5)
- new net DTR: Q1.1 (G), Q2.2 (S), R1.1, U2.23 (DTR)
- new net EN: SW2.2 (B), U11.3 (EN)
- new net GND: C1.2, C10.2, C11.2, C12.2, C13.2, C14.2, C15.2, C16.2, C17.2, C18.2, C19.2, C2.2, C20.2, C21.2, C23.2, C24.2, C25.2, C26.2, C27.2, C28.2, C29.2, C3.2, C4.2, C5.2, C7.2, C9.2, D1.2 (GND), D5.2 (A), D6.1 (K), D9.1 (K), DS1.1 (GND), DS1.12 (GND), DS1.5 (GND), DS1.6 (GND), DS1.8 (nCS), J1.A1 (GND), J1.A12 (GND), J1.B1 (GND), J1.B12 (GND), J1.S1 (SHIELD), J2.S, J4.11 (SHIELD), J4.6 (VSS), J5.1 (Pin_1), Q3.2 (S), Q5.2 (S), R1.2, R12.2, R16.2, R2.2, R21.2, R25.2, R30.2, R33.2, R34.2, R35.2, R37.2, R38.2, R4.2, R40.2, R5.2, R9.2, SW1.2, SW2.1 (A), U1.2 (V-), U10.5 (RES), U10.6 (GND), U10.7 (GND), U10.8 (GND), U11.2 (GND), U2.2 (GND), U2.25 (GND), U3.2 (VSS), U4.2 (GND), U5.2 (GND), U6.6 (GND), U6.8 (GND), U7.6 (S2), U8.23 (VSS), U8.35 (VSS), U8.47 (VSS), U8.49 (PAD), U8.8 (VSSA/VREF-), U9.4 (GND), VR1.3 (X-), VR1.6 (-Y)
- new net I2C1_SCL: J5.9 (Pin_9), R27.2, U10.1 (SCL/SPC), U8.42 (PB6)
- new net I2C1_SDA: J5.11 (Pin_11), R28.2, U10.4 (SDA/SDI), U8.43 (PB7)
- new net IR_RX: U6.3 (OUT), U8.20 (PB2)
- new net IR_TX: R18.1, U8.46 (PB9)
- new net JOY_X: U8.13 (PA3), VR1.2 (X)
- new net JOY_Y: U8.14 (PA4), VR1.5 (Y)
- new net LCD_DC: DS1.7 (D/C), U8.33 (PA12)
- new net LCD_LED: Q5.1 (G), R30.1, U8.45 (PB8)
- new net LCD_MOSI: DS1.10 (SDA), U8.41 (PB5)
- new net LCD_RESET: DS1.11 (nRESET), U8.40 (PB4)
- new net LCD_SCK: DS1.9 (SCL), U8.39 (PB3)
- new net LEDK: DS1.2 (LEDK), R31.1
- new net LEDK2: Q5.3 (D), R31.2
- new net LED_B: R22.2, U8.11 (PA1)
- new net LED_CHG: D4.2 (A), R14.2
- new net LED_G: R23.2, U8.32 (PA11)
- new net LED_PWR: D9.2 (A), R32.2
- new net LED_R: R24.1, U8.29 (PA8)
- new net LED_RX: D2.2 (A), D5.1 (K), R11.2, U6.7 (IN)
- new net LED_TX: D3.2 (A), D6.2 (A), R13.2, R18.2
- new net PROG: R16.1, U3.5 (PROG)
- new net QSPI_CLK: U8.21 (PB10), U9.6 (CLK)
- new net QSPI_IO0: U8.19 (PB1), U9.5 (IO0)
- new net QSPI_IO1: U8.18 (PB0), U9.2 (IO1)
- new net QSPI_IO2: U8.17 (PA7), U9.3 (IO2)
- new net QSPI_IO3: U8.16 (PA6), U9.7 (IO3)
- new net QSPI_NCS: R26.2, U8.22 (PB11), U9.1 (nCS)
- new net RESET: C4.1, J5.3 (Pin_3), Q2.3 (D), R7.2, SW1.1, U8.7 (NRST)
- new net RGB_B: D7.4 (BK), R22.1
- new net RGB_G: D7.3 (GK), R23.1
- new net RGB_R: D7.2 (RK), R24.2
- new net RTS: Q1.2 (S), Q2.1 (G), R2.1, U2.19 (RTS)
- new net RXT: D2.1 (K), U2.13 (GPIO1/RXT)
- new net SPEAKER_+: LS1.1, U4.6 (OUT+)
- new net SPEAKER_-: LS1.2, U4.1 (OUT-)
- new net SPI2_MISO: J4.7 (DAT0), J5.6 (Pin_6), U8.27 (PB14)
- new net SPI2_MOSI: J4.3 (CMD), J5.8 (Pin_8), U8.28 (PB15)
- new net SPI2_NSS: J4.2 (DAT3/CD), R29.2, U8.25 (PB12)
- new net SPI2_SCK: J4.5 (CLK), J5.4 (Pin_4), U8.26 (PB13)
- new net STM32_CLK: U5.3 (OUT), U8.5 (PH0/OSC_IN)
- new net STM32_RX: R19.2, U2.21 (TXD), U8.31 (PA10)
- new net STM32_TX: R17.2, U2.20 (RXD), U8.30 (PA9)
- new net SWCLK: J5.5 (Pin_5), U8.37 (PA14)
- new net SWDIO: J5.7 (Pin_7), U8.34 (PA13)
- new net TXT: D3.1 (K), U2.14 (GPIO0/TXT)
- new net USART2_RX: J5.12 (Pin_12), U8.38 (PA15)
- new net USART2_TX: J5.10 (Pin_10), U8.12 (PA2)
- new net USB_DM: D1.3 (IO2), J1.A7 (D-), J1.B7 (D-), U2.4 (D-)
- new net USB_DP: D1.4 (IO3), J1.A6 (D+), J1.B6 (D+), U2.3 (D+)
- new net USB_RST: R3.2, U2.9 (RSTb)
- new net VBAT: C14.1, J3.1 (+), Q4.3 (D), R20.1, U3.3 (VBAT)
- new net VCC: C16.1, C18.1, C26.1, D8.1 (K), Q4.2 (S), R39.1, SW2.3 (C), U11.1 (IN), U4.5 (VDD)
- new net VCC_DET: R39.2, R40.1, U8.10 (PA0)
- new net VM: R21.1, U7.5 (VM)
- new net VUSB: C7.1, D1.1 (IO1), D8.2 (A), J1.A4 (VBUS), J1.A9 (VBUS), J1.B4 (VBUS), J1.B9 (VBUS), Q4.1 (G), R14.1, R25.1, R36.1, U3.4 (VDD)
- new net VUSB_DET: R36.2, R37.1, U2.8 (VBUS)
- no-connect marks 0 -> 26
Other:
- note added: "15mA\n1.1V"
- note added: "1\n2\n3\n4\n5\n6\n7\n8\n9\n10\n11\n12"
- note added: "200mA Max."
- note added: "25mcd\n0.6mA\n2.4V"
- note added: "25mcd\n1.4mA\n1.9V"
- note added: "25mcd\n2.5mA\n2.7V"
- note added: "3V3 Regulator"
- note added: "5mcd\n0.5mA\n2.4V"
- note added: "5mcd\n1.3mA\n1.8V"
- note added: "5mcd\n2.5mA\n2.0V"
- note added: "Accelerometer"
- note added: "Audio Output"
- note added: "BOOT0\n\n0\n0\n0\n1"
- note added: "Battery Charger"
- note added: "Battery Protection"
- note added: "Controller"
- note added: "DTR\n\n0\n1\n0\n1"
- note added: "Display"
- note added: "Expansion Port"
- note added: "Flash Memory"
- note added: "GND\n3V3 (OUTPUT ONLY)\nRESET (ACTIVE LOW)\nSPI2_SCK\nGPIO (PA14) / SWCLK\nSPI2_MISO\nGPIO (PA13) / SWDIO\nSPI2_MOSI\nI2C1_SCL\nGPIO (PA2) / ADC1_IN7 / USART2_TX\nI2C1_SDA\nGPIO (PA15) / USART2_RX\n"
- note added: "IR Interface"
- note added: "IREG\n50mA"
- note added: "Microcontroller"
- note added: "Note: For more details open the file audio-simulation.asc in LTspice"
- note added: "RESET\n\n1\n1\n0\n1"
- note added: "RGB LED"
- note added: "RTS\n\n0\n1\n1\n0"
- note added: "Reset and Boot Mode Selector"
- note added: "USB Type-C Interface"
- note added: "USB<->USART Bridge"
- note added: "Voltage Dividers"
- note added: "Warning:\n- I2C1 is shared with on-board accelerometer.\n- SPI2 is shared with on-board microSD socket. Use a GPIO as CS.\n- Maximum current per pin is 20mA.\n- Total maximum current (including on-board components) is 200mA.\n- Never exceed total maximum current when running on battery!!!"
- note added: "Warning:\n- Use rechargeable LIR2450 only.\n- Non-rechargeable CR2450 is prohibited.\n- Insert battery with correct polarity only.\n- Reverse polarity will cause damage.\n"
- note added: "microSD Card"

Commit message: PCB v0.2: Reduced component dimensions. Preliminary placement
Parts:
- removed LS1: CMS-151135-078S, _AKL_Speaker:Speaker_15x11mm, symbol _AKL_Speaker:CMS-151135-078S
- removed SW1: RESET, _AKL_Switch:EVQPU, symbol _AKL_Switch:EVQ-PUL02K
- removed SW5: START, _AKL_Switch:EVQPU, symbol _AKL_Switch:EVQ-PUL02K
- removed SW6: SELECT, _AKL_Switch:EVQPU, symbol _AKL_Switch:EVQ-PUL02K
- added LS1: CMS-151125-078S, _AKL_Speaker:Speaker_15x11mm, symbol _AKL_Speaker:CMS-151125-078S
- added SW1: RESET, _AKL_Switch:EVQP7, symbol _AKL_Switch:EVQ-P7L01P
- added SW5: START, _AKL_Switch:EVQP7, symbol _AKL_Switch:EVQ-P7L01P
- added SW6: SELECT, _AKL_Switch:EVQP7, symbol _AKL_Switch:EVQ-P7L01P
- C1, C13, C14, C17, C20, C23, C26, C28, C7: footprint Capacitor_SMD:C_0805_2012Metric -> Capacitor_SMD:C_0603_1608Metric; MPN CL21A106KOQNNNG -> CL10A106KP8NNNC
- C10, C16, C9: footprint Capacitor_SMD:C_0603_1608Metric -> Capacitor_SMD:C_0402_1005Metric; MPN CL10B105KA8NNNC -> CL05A105KO5NNNC
- C11, C12, C15, C19, C2, C21, C22, C24, C25, C27, C29, C3, C4, C5, C8: footprint Capacitor_SMD:C_0603_1608Metric -> Capacitor_SMD:C_0402_1005Metric; MPN CL10B104KB8NNNL -> CL05B104KO5NNNC
- C18, C6: MPN CL32A107MQVNNWE -> CL32A107MQVNNNE
- J1: footprint Connector_USB:USB_C_Receptacle_HRO_TYPE-C-31-M-12 -> _AKL_Connector:TYPE-C-31-M-12
- J4: footprint Connector_Card:microSD_HC_Molex_104031-0811 -> _AKL_Connector:1040310811
- Q1, Q2, Q3, Q5: value FDN327N -> SI2102-TP; footprint Package_TO_SOT_SMD:SOT-23 -> Package_TO_SOT_SMD:SOT-323_SC-70; symbol _AKL_Transistor:FDN327N -> _AKL_Transistor:SI2102-TP; MPN FDN327N -> SI2102-TP
- Q4: value FDN340P -> SI2101-TP; footprint Package_TO_SOT_SMD:SOT-23 -> Package_TO_SOT_SMD:SOT-323_SC-70; symbol _AKL_Transistor:FDN340P -> _AKL_Transistor:SI2101-TP; MPN FDN340P -> SI2101-TP
- R1, R10, R16, R2, R26, R29, R30, R33, R34, R35, R38, R6, R7: footprint Resistor_SMD:R_0603_1608Metric -> Resistor_SMD:R_0402_1005Metric; symbol _AKL_Resistor:20K -> _AKL_Resistor_402:20K; MPN RC0603FR-0720KL -> RC0402FR-0720KL
- R11, R12, R13, R23: footprint Resistor_SMD:R_0603_1608Metric -> Resistor_SMD:R_0402_1005Metric; symbol _AKL_Resistor:1K8 -> _AKL_Resistor_402:1K8; MPN RC0603FR-071K8L -> RC0402FR-071K8L
- R14, R21: footprint Resistor_SMD:R_0603_1608Metric -> Resistor_SMD:R_0402_1005Metric; symbol _AKL_Resistor:2K4 -> _AKL_Resistor_402:2K4; MPN RC0603FR-072K4L -> RC0402FR-072K4L
- R15, R25, R37, R40: footprint Resistor_SMD:R_0603_1608Metric -> Resistor_SMD:R_0402_1005Metric; symbol _AKL_Resistor:120K -> _AKL_Resistor_402:120K; MPN RC0603FR-07120KL -> RC0402FR-07120KL
- R17, R19, R27, R28, R4, R5: footprint Resistor_SMD:R_0603_1608Metric -> Resistor_SMD:R_0402_1005Metric; symbol _AKL_Resistor:5K1 -> _AKL_Resistor_402:5K1; MPN RC0603FR-075K1L -> RC0402FR-075K1L
- R18: footprint Resistor_SMD:R_0603_1608Metric -> Resistor_SMD:R_0402_1005Metric; symbol _AKL_Resistor:150 -> _AKL_Resistor_402:150; MPN RC0603FR-07150RL -> RC0402FR-07150RL
- R20, R32: footprint Resistor_SMD:R_0603_1608Metric -> Resistor_SMD:R_0402_1005Metric; symbol _AKL_Resistor:510 -> _AKL_Resistor_402:510; MPN RC0603FR-07510RL -> RC0402FR-07510RL
- R22, R8: footprint Resistor_SMD:R_0603_1608Metric -> Resistor_SMD:R_0402_1005Metric; symbol _AKL_Resistor:240 -> _AKL_Resistor_402:240; MPN RC0603FR-07240RL -> RC0402FR-07240RL
- R24, R3: footprint Resistor_SMD:R_0603_1608Metric -> Resistor_SMD:R_0402_1005Metric; symbol _AKL_Resistor:1K -> _AKL_Resistor_402:1K; MPN RC0603FR-071KL -> RC0402FR-071KL
- R31, R9: footprint Resistor_SMD:R_0603_1608Metric -> Resistor_SMD:R_0402_1005Metric; symbol _AKL_Resistor:100 -> _AKL_Resistor_402:100; MPN RC0603FR-0710RL -> RC0402FR-07100RL
- R36, R39: footprint Resistor_SMD:R_0603_1608Metric -> Resistor_SMD:R_0402_1005Metric; symbol _AKL_Resistor:75K -> _AKL_Resistor_402:75K; MPN RC0603FR-0775KL -> RC0402FR-0775KL
- U1: value TLV9061IDBVR -> TLV9061IDCKR; footprint Package_TO_SOT_SMD:SOT-23-5 -> Package_TO_SOT_SMD:SOT-353_SC-70-5; symbol _AKL_IC:TLV9061IDBVR -> _AKL_IC:TLV9061IDCKR; MPN TLV9061IDBVR -> TLV9061IDCKR
- U10: footprint Package_LGA:LGA-12_2x2mm_P0.5mm -> _AKL_IC:LIS2DE12TR
- U9: footprint Package_SON:WSON-8-1EP_6x5mm_P1.27mm_EP3.4x4.3mm -> _AKL_IC:Winbond_WSON8_6x5mm
Connections:
- net 3V3: now also SW5.1, SW6.1
- net AUD1: now also U1.3 (-); no longer U1.1
- net BTN_SELECT: now also SW6.2
- net BTN_START: now also SW5.2
- net DAC_PWM_OUT: now also U1.1 (+); no longer U1.3 (+)
- net GND: now also SW1.2
- net RESET: now also SW1.1
- net SPEAKER_+: now also LS1.1
- net SPEAKER_-: now also LS1.2
Other:
- moved on the sheet: R22, R24, VR1

Commit message: PCB v0.2: Starting to route
Parts:
- D8: value MBR0520L -> NSR0520V2T1G; footprint Diode_SMD:D_SOD-123 -> Diode_SMD:D_SOD-523; symbol _AKL_Diode:MBR0520L -> _AKL_Diode:NSR0520V2T1G; MPN MBR0520L -> NSR0520V2T1G
- J3: value BK-880 -> Battery; footprint _AKL_Battery:BK-880 -> _AKL_Battery:Solder_Pad_D2; symbol _AKL_Battery:BK-880 -> _AKL_Battery:Solder_Pad_D2
Other:
- note removed: "Warning:\n- Use rechargeable LIR2450 only.\n- Non-rechargeable CR2450 is prohibited.\n- Insert battery with correct polarity only.\n- Reverse polarity will cause damage.\n"
- moved on the sheet: C22, J3, R20, R21, U7
Changed lines of the file:
@@
 Sheet 1 1
 Title "OpenHandheld MX"
-Date "2020-04-26"
+Date "2020-06-19"
 Rev "v0.2"
 Comp "The OpenHandheld Project"
@@
 L power:GND #PWR043
 U 1 1 5E7FFD2B
-P 9750 1950
-F 0 "#PWR043" H 9750 1700 50  0001 C CNN
-F 1 "GND" H 9750 1800 50  0000 C CNN
-F 2 "" H 9750 1950 50  0001 C CNN
-F 3 "" H 9750 1950 50  0001 C CNN
-	1    9750 1950
+P 9700 2200
+F 0 "#PWR043" H 9700 1950 50  0001 C CNN
+F 1 "GND" H 9700 2050 50  0000 C CNN
+F 2 "" H 9700 2200 50  0001 C CNN
+F 3 "" H 9700 2200 50  0001 C CNN
+	1    9700 2200
 	1    0    0    -1
 $EndComp
@@
 Text Label 6750 1300 2    50   ~ 0
 VBAT
-Wire Notes Line
-	7450 2050 9200 2050
-Wire Notes Line
-	7450 2550 7450 2050
-Wire Notes Line
-	9200 2550 7450 2550
-Wire Notes Line
-	9200 2050 9200 2550
-Text Notes 7500 2500 0    50   ~ 0
-Warning:\n- Use rechargeable LIR2450 only.\n- Non-rechargeable CR2450 is prohibited.\n- Insert battery with correct polarity only.\n- Reverse polarity will cause damage.\n
 Text Notes 4200 850  0    79   Italic 16
 Battery Charger
@@
 	11800 1700 11800 1500
 $Comp
-L _AKL_Battery:BK-880 J3
+L _AKL_Battery:Solder_Pad_D2 J3
 U 1 1 5E8574BB
-P 7900 1500
-F 0 "J3" H 8018 1596 50  0000 L CNN
-F 1 "BK-880" H 8018 1505 50  0000 L CNN
-F 2 "_AKL_Battery:BK-880" V 7900 1560 50  0001 C CNN
-F 3 "https://www.digikey.es/product-detail/es/mpd-memory-protection-devices/BK-880/BK-880-ND/2439467" V 7900 1560 50  0001 C CNN
-F 4 "BK-880" H 7900 1500 50  0001 C CNN "MPN"
-	1    7900 1500
+P 7850 1750
+F 0 "J3" H 7968 1846 50  0000 L CNN
+F 1 "Battery" H 7968 1755 50  0000 L CNN
+F 2 "_AKL_Battery:Solder_Pad_D2" V 7850 1810 50  0001 C CNN
+F 3 "https://www.digikey.es/product-detail/es/mpd-memory-protection-devices/BK-880/BK-880-ND/2439467" V 7850 1810 50  0001 C CNN
+F 4 "BK-880" H 7850 1750 50  0001 C CNN "MPN"
+	1    7850 1750
 	1    0    0    -1
 $EndComp
@@
 	1    0    0    -1
 $EndComp
-NoConn ~ 9250 1850
-NoConn ~ 9600 1500
+NoConn ~ 9200 2100
+NoConn ~ 9550 1750
 Wire Wire Line
-	9400 1850 9400 1900
+	9350 2100 9350 2150
 Wire Wire Line
-	9600 1350 9750 1350
+	9550 1600 9700 1600
 Wire Wire Line
-	9750 1350 9750 1400
+	9700 1600 9700 1650
 Wire Wire Line
-	9750 1700 9750 1900
+	9700 1950 9700 2150
 Wire Wire Line
-	9750 1900 9400 1900
+	9700 2150 9350 2150
 $Comp
 L _AKL_Capacitor:100nF C22
 U 1 1 5E9CB7D4
-P 8450 1600
-F 0 "C22" H 8565 1646 50  0000 L CNN
-F 1 "100nF" H 8565 1555 50  0000 L CNN
-F 2 "Capacitor_SMD:C_0402_1005Metric" H 8488 1450 50  0001 C CNN
-F 3 "https://www.digikey.es/product-detail/es/samsung-electro-mechanics/CL05B104KO5NNNC/1276-1001-1-ND/3889087" H 8450 1600 50  0001 C CNN
-F 4 "CL05B104KO5NNNC" H 8450 1600 50  0001 C CNN "MPN"
-	1    8450 1600
+P 8400 1850
+F 0 "C22" H 8515 1896 50  0000 L CNN
+F 1 "100nF" H 8515 1805 50  0000 L CNN
+F 2 "Capacitor_SMD:C_0402_1005Metric" H 8438 1700 50  0001 C CNN
+F 3 "https://www.digikey.es/product-detail/es/samsung-electro-mechanics/CL05B104KO5NNNC/1276-1001-1-ND/3889087" H 8400 1850 50  0001 C CNN
+F 4 "CL05B104KO5NNNC" H 8400 1850 50  0001 C CNN "MPN"
+	1    8400 1850
 	1    0    0    -1
 $EndComp
 Wire Wire Line
-	8450 1750 8450 1900
+	8400 2000 8400 2150
 Wire Wire Line
-	8450 1900 8850 1900
+	8400 2150 8800 2150
 Wire Wire Line
-	9100 1900 9100 1850
+	9050 2150 9050 2100
 Wire Wire Line
-	8450 1300 8450 1350
+	8400 1550 8400 1600
 Wire Wire Line
-	8450 1350 8900 1350
-Connection ~ 8450 1350
+	8400 1600 8850 1600
+Connection ~ 8400 1600
 Wire Wire Line
-	8450 1350 8450 1450
+	8400 1600 8400 1700
 Wire Wire Line
-	8900 1500 8850 1500
+	8850 1750 8800 1750
 Wire Wire Line
-	8850 1500 8850 1900
-Connection ~ 8850 1900
+	8800 1750 8800 2150
+Connection ~ 8800 2150
 Wire Wire Line
-	8850 1900 9100 1900
-Connection ~ 8450 1900
+	8800 2150 9050 2150
+Connection ~ 8400 2150
 Wire Wire Line
-	8450 950  8450 1000
-Text Label 9900 950  2    50   ~ 0
+	8400 1200 8400 1250
+Text Label 9850 1200 2    50   ~ 0
 VBAT
 Wire Wire Line
-	7900 1300 7900 950
+	7850 1550 7850 1200
 Wire Wire Line
-	7900 950  8450 950
+	7850 1200 8400 1200
 Wire Wire Line
-	7900 1600 7900 1900
+	7850 1850 7850 2150
 Wire Wire Line
-	7900 1900 8450 1900
+	7850 2150 8400 2150
 Wire Wire Line
-	9750 1900 9750 1950
-Connection ~ 9750 1900
-Connection ~ 8450 950
+	9700 2150 9700 2200
+Connection ~ 9700 2150
+Connection ~ 8400 1200
 $Comp
 L _AKL_Resistor_402:2K4 R21
 U 1 1 5EA90202
-P 9750 1550
-F 0 "R21" H 9820 1596 50  0000 L CNN
-F 1 "2K4" H 9820 1505 50  0000 L CNN
-F 2 "Resistor_SMD:R_0402_1005Metric" H 9750 1550 50  0001 C CNN
-F 3 "https://www.digikey.es/product-detail/es/yageo/RC0402FR-072K4L/311-2-40KLRCT-ND/729502" H 9750 1550 50  0001 C CNN
-F 4 "RC0402FR-072K4L" H 9750 1550 44  0001 C CNN "MPN"
-	1    9750 1550
+P 9700 1800
+F 0 "R21" H 9770 1846 50  0000 L CNN
+F 1 "2K4" H 9770 1755 50  0000 L CNN
+F 2 "Resistor_SMD:R_0402_1005Metric" H 9700 1800 50  0001 C CNN
+F 3 "https://www.digikey.es/product-detail/es/yageo/RC0402FR-072K4L/311-2-40KLRCT-ND/729502" H 9700 1800 50  0001 C CNN
+F 4 "RC0402FR-072K4L" H 9700 1800 44  0001 C CNN "MPN"
+	1    9700 1800
 	1    0    0    -1
 $EndComp
@@
 	11400 1500 11400 1350
 $Comp
-L _AKL_Diode:MBR0520L D8
+L _AKL_Diode:NSR0520V2T1G D8
 U 1 1 5EC15C97
 P 11100 1500
-F 0 "D8" H 11100 1600 50  0000 C CNN
-F 1 "MBR0520L" H 11100 1400 50  0000 C CNN
-F 2 "Diode_SMD:D_SOD-123" H 11100 1500 50  0001 C CNN
-F 3 "https://www.digikey.es/product-detail/es/on-semiconductor/MBR0520L/MBR0520LCT-ND/458961" H 11100 1500 50  0001 C CNN
-F 4 "MBR0520L" H 11100 1500 50  0001 C CNN "MPN"
+F 0 "D8" H 11100 1400 50  0000 C CNN
+F 1 "NSR0520V2T1G" H 11100 1600 50  0000 C CNN
+F 2 "Diode_SMD:D_SOD-523" H 11100 1500 50  0001 C CNN
+F 3 "https://www.digikey.es/product-detail/es/on-semiconductor/NSR0520V2T1G/NSR0520V2T1GOSCT-ND/1981501" H 11100 1500 50  0001 C CNN
+F 4 "NSR0520V2T1G" H 11100 1500 50  0001 C CNN "MPN"
 	1    11100 1500
 	-1   0    0    1
@@
 L _AKL_IC:AP9211S-AN-HAC-7 U7
 U 1 1 5F172420
-P 9250 1500
-F 0 "U7" H 9250 1915 50  0000 C CNN
-F 1 "AP9211S-AN-HAC-7" H 9250 1824 50  0000 C CNN
-F 2 "_AKL_IC:AP9211S-AN-HAC-7" H 8950 2450 50  0001 C CNN
-F 3 "https://www.mouser.es/ProductDetail/Diodes-Incorporated/AP9211S-AN-HAC-7?qs=%2Fha2pyFaduhU8ORG8s%252BdQ8wjonur7%2FvJn%252BxxLU0AZ5qESSeNUE%2F1LA%3D%3D" H 8950 2450 50  0001 C CNN
-F 4 "AP9211S-AN-HAC-7" H 9250 1800 50  0001 C CNN "MPN"
-	1    9250 1500
+P 9200 1750
+F 0 "U7" H 9200 2165 50  0000 C CNN
+F 1 "AP9211S-AN-HAC-7" H 9200 2074 50  0000 C CNN
+F 2 "_AKL_IC:AP9211S-AN-HAC-7" H 8900 2700 50  0001 C CNN
+F 3 "https://www.mouser.es/ProductDetail/Diodes-Incorporated/AP9211S-AN-HAC-7?qs=%2Fha2pyFaduhU8ORG8s%252BdQ8wjonur7%2FvJn%252BxxLU0AZ5qESSeNUE%2F1LA%3D%3D" H 8900 2700 50  0001 C CNN
+F 4 "AP9211S-AN-HAC-7" H 9200 2050 50  0001 C CNN "MPN"
+	1    9200 1750
 	1    0    0    -1
 $EndComp
@@
 L _AKL_Resistor_402:510 R20
 U 1 1 5EBDA8F2
-P 8450 1150
-F 0 "R20" H 8520 1196 50  0000 L CNN
-F 1 "510" H 8520 1105 50  0000 L CNN
-F 2 "Resistor_SMD:R_0402_1005Metric" H 8450 1150 50  0001 C CNN
-F 3 "https://www.digikey.es/product-detail/es/yageo/RC0402FR-07510RL/311-510LRCT-ND/729579" H 8450 1150 50  0001 C CNN
-F 4 "RC0402FR-07510RL" H 8450 1150 44  0001 C CNN "MPN"
-	1    8450 1150
+P 8400 1400
+F 0 "R20" H 8470 1446 50  0000 L CNN
+F 1 "510" H 8470 1355 50  0000 L CNN
+F 2 "Resistor_SMD:R_0402_1005Metric" H 8400 1400 50  0001 C CNN
+F 3 "https://www.digikey.es/product-detail/es/yageo/RC0402FR-07510RL/311-510LRCT-ND/729579" H 8400 1400 50  0001 C CNN
+F 4 "RC0402FR-07510RL" H 8400 1400 44  0001 C CNN "MPN"
+	1    8400 1400
 	1    0    0    -1
 $EndComp
 Wire Wire Line
-	8450 950  9900 950
+	8400 1200 9850 1200
 Text Notes 750  10950 0    50   ~ 0
 Note: For more details open the file audio-simulation.asc in LTspice
@@
 Text Label 6150 1450 0    50   ~ 0
 PROG
-Text Label 7900 1900 0    50   ~ 0
+Text Label 7850 2150 0    50   ~ 0
 BAT_GND
-Text Label 8450 1450 0    50   ~ 0
+Text Label 8400 1700 0    50   ~ 0
 AP9_VDD
-Text Label 9600 1350 0    50   ~ 0
+Text Label 9550 1600 0    50   ~ 0
 VM
 Text Label 12250 1800 0    50   ~ 0

Commit message: PCB v0.2: Finished placement, created power planes
Connections:
- net USB_DM: now also D1.4 (IO3); no longer D1.3 (IO2)
- net USB_DP: now also D1.3 (IO2); no longer D1.4 (IO3)
Changed lines of the file:
@@
 $EndComp
-Wire Wire Line
-	2950 1450 3600 1450
-Wire Wire Line
-	2850 1250 3600 1250
 Wire Wire Line
 	2750 1150 3600 1150
-Connection ~ 2950 1450
-Wire Wire Line
-	2950 1700 2950 1450
-Connection ~ 2850 1250
-Wire Wire Line
-	2850 1700 2850 1250
 Connection ~ 2750 1150
 Wire Wire Line
 	2750 1700 2750 1150
 Wire Wire Line
-	1950 1450 2950 1450
-Wire Wire Line
-	1950 1250 2850 1250
+	1950 1450 2850 1450
 Wire Wire Line
 	1900 1150 2750 1150
@@
 	1    0    0    -1
 $EndComp
+Wire Wire Line
+	1950 1250 2950 1250
+Wire Wire Line
+	2850 1700 2850 1450
+Connection ~ 2850 1450
+Wire Wire Line
+	2850 1450 3600 1450
+Wire Wire Line
+	2950 1700 2950 1250
+Connection ~ 2950 1250
+Wire Wire Line
+	2950 1250 3600 1250
 $EndSCHEMATC

Commit message: PCB v0.2: STM32 fanout
Connections:
- net JOY_X: now also U8.14 (PA4); no longer U8.13 (PA3)
- net JOY_Y: now also U8.13 (PA3); no longer U8.14 (PA4)
- net LED_RX: no longer D2.2 (A), R11.2
- net LED_TX: no longer D3.2 (A), R13.2
- new net LED_RXD: D2.2 (A), R11.2
- new net LED_TXD: D3.2 (A), R13.2
Changed lines of the file:
@@
 Text Label 15200 3750 0    50   ~ 0
 USART2_TX
+Text Label 9300 5700 3    50   ~ 0
+JOY_X
 Text Label 9200 5700 3    50   ~ 0
-JOY_X
-Text Label 9300 5700 3    50   ~ 0
 JOY_Y
 Text Label 9400 5700 3    50   ~ 0
@@
 USB_RST
 Text Label 3900 4500 0    50   ~ 0
-LED_RX
+LED_RXD
 Text Label 4350 4500 0    50   ~ 0
-LED_TX
+LED_TXD
 Text Label 3600 4850 0    50   ~ 0
 RXT

Commit message: PCB v0.2: Silkscreen.
Parts:
- SW3: value A -> B
- SW4: value B -> A
Connections:
- net BTN_A: now also R34.1, SW4.1, U8.3 (PC14/OSC32_IN); no longer R33.1, SW3.1, U8.2 (PC13)
- net BTN_B: now also R33.1, SW3.1, U8.2 (PC13); no longer R34.1, SW4.1, U8.3 (PC14/OSC32_IN)
Changed lines of the file:
@@
 Text Label 15200 3650 0    50   ~ 0
 SPI2_MOSI
-Text Label 9900 3400 1    50   ~ 0
+Text Label 10000 3400 1    50   ~ 0
 BTN_A
-Text Label 10000 3400 1    50   ~ 0
-BTN_B
 Text Label 10100 3400 1    50   ~ 0
 BTN_START
@@
 P 13800 7100
 F 0 "SW3" V 13850 7300 50  0000 C CNN
-F 1 "A" V 13750 7300 50  0000 C CNN
+F 1 "B" V 13750 7300 50  0000 C CNN
 F 2 "_AKL_Switch:TL3301TF160QG" H 13800 7300 50  0001 C CNN
 F 3 "https://www.digikey.es/product-detail/es/e-switch/TL3301TF160QG/TL3301TF160QGCT-ND/4835081" H 13800 7300 50  0001 C CNN
@@
 P 14250 7100
 F 0 "SW4" V 14300 7300 50  0000 C CNN
-F 1 "B" V 14200 7300 50  0000 C CNN
+F 1 "A" V 14200 7300 50  0000 C CNN
 F 2 "_AKL_Switch:TL3301TF160QG" H 14250 7300 50  0001 C CNN
 F 3 "https://www.digikey.es/product-detail/es/e-switch/TL3301TF160QG/TL3301TF160QGCT-ND/4835081" H 14250 7300 50  0001 C CNN
@@
 $EndComp
 Text Label 13800 7350 0    50   ~ 0
+BTN_B
+Text Label 14250 7350 0    50   ~ 0
 BTN_A
-Text Label 14250 7350 0    50   ~ 0
-BTN_B
 Text Label 14700 7350 0    50   ~ 0
 BTN_START
@@
 Wire Wire Line
 	2950 1250 3600 1250
+Text Label 9900 3400 1    50   ~ 0
+BTN_B
 $EndSCHEMATC

Commit message: Case v0.2: Finished
Parts:
- J3: MPN BK-880 -> (none)
Changed lines of the file:
@@
 F 1 "Battery" H 7968 1755 50  0000 L CNN
 F 2 "_AKL_Battery:Solder_Pad_D2" V 7850 1810 50  0001 C CNN
-F 3 "https://www.digikey.es/product-detail/es/mpd-memory-protection-devices/BK-880/BK-880-ND/2439467" V 7850 1810 50  0001 C CNN
-F 4 "BK-880" H 7850 1750 50  0001 C CNN "MPN"
+F 3 "" V 7850 1810 50  0001 C CNN
+F 4 "" H 7850 1750 50  0001 C CNN "MPN"
 	1    7850 1750
 	1    0    0    -1
